Commit message: Update cma_urdf.xacro
With vacuum gripper

File: cma_urdf.xacro (robot description, xacro)
@@ -172,5 +172,5 @@
       <origin rpy="0 0 0" xyz="-0.4826 -0.0744 -1.12545"/>
       <geometry>
-        <mesh filename="package://cma_urdf_description/meshes/Link6_UR5_1.stl" scale="0.001 0.001 0.001"/>
+        <mesh filename="package://cma_urdf_description/meshes/Link6_UR5_1_and_VG10.stl" scale="0.001 0.001 0.001"/>
       </geometry>
       <material name="silver"/>
@@ -179,8 +179,344 @@
       <origin rpy="0 0 0" xyz="-0.4826 -0.0744 -1.12545"/>
       <geometry>
-        <mesh filename="package://cma_urdf_description/meshes/Link6_UR5_1.stl" scale="0.001 0.001 0.001"/>
-      </geometry>
-    </collision>
-  </link>
+        <mesh filename="package://cma_urdf_description/meshes/Link6_UR5_1_and_VG10.stl" scale="0.001 0.001 0.001"/>
+      </geometry>
+    </collision>
+  </link>
+      <joint name="${prefix}ee_fixed_joint" type="fixed">
+      <parent link="${prefix}Link6_UR5_1" />
+      <child link = "${prefix}ee_link" />
+      <origin xyz="0.0 ${wrist_3_length} 0.0" rpy="0.0 0.0 ${pi/2.0}" />
+    </joint>
+    <link name="${prefix}ee_link">
+      <collision>
+        <geometry>
+          <box size="0.01 0.01 0.01"/>
+        </geometry>
+        <surface>
+          <friction>
+            <ode>
+              <mu>10</mu>
+              <mu2>10</mu2>
+            </ode>
+          </friction>
+        </surface>
+        <origin rpy="0 0 0" xyz="-0.01 0 0"/>
+      </collision>
+    </link>
+    <link name="vacuum_gripper">
+      <gravity>0</gravity>
+      <visual>
+        <origin rpy="0 0 0" xyz="0 0 0"/>
+        <geometry>
+          <cylinder radius="0.005" length="0.01"/>
+        </geometry>
+        <material name="transparent">
+          <color rgba="0 0 0 0"/>
+        </material>
+      </visual>
+      <inertial>
+        <origin rpy="0 0 0" xyz="0.000000 0.000000 0.000000"/>
+        <mass value="0.0001"/>
+        <inertia ixx="1e-08" ixy="0" ixz="0" iyy="1e-08" iyz="0" izz="1e-08"/>
+      </inertial>
+    </link>
+    <joint name="gripper_joint" type="revolute">
+      <axis xyz="1 0 0" />
+      <parent link="ee_link" />
+      <child link="vacuum_gripper" />
+      <origin rpy="0 1.5708 0" xyz="0.01 0.0125 0" />
+      <limit effort="50" velocity="50" lower="0" upper="0" />
+      <dynamics damping="0.0" friction="10"/>
+    </joint>
+  <gazebo>
+      <plugin name="gazebo_ros_vacuum_gripper" filename="libgazebo_ros_vacuum_gripper.so">
+        <robotNamespace>/ur5/vacuum_gripper</robotNamespace>
+        <bodyName>vacuum_gripper</bodyName>
+        <topicName>grasping</topicName>
+	<maxForce>50</maxForce>
+        <maxDistance>0.05</maxDistance>
+        <minDistance>0.01</minDistance>
+      </plugin>
+  </gazebo>
+    <link name="vacuum_gripper1">
+      <gravity>0</gravity>
+      <visual>
+        <origin rpy="0 0 0" xyz="0 0 0"/>
+        <geometry>
+          <cylinder radius="0.005" length="0.01"/>
+        </geometry>
+        <material name="transparent">
+          <color rgba="0 0 0 0"/>
+        </material>
+      </visual>
+      <inertial>
+        <origin rpy="0 0 0" xyz="0.000000 0.000000 0.000000"/>
+        <mass value="0.0001"/>
+        <inertia ixx="1e-08" ixy="0" ixz="0" iyy="1e-08" iyz="0" izz="1e-08"/>
+      </inertial>
+    </link>
+    <joint name="gripper_joint1" type="revolute">
+      <axis xyz="1 0 0" />
+      <parent link="ee_link" />
+      <child link="vacuum_gripper1" />
+      <origin rpy="0 1.5708 0" xyz="0.01 -0.0125 0" />
+      <limit effort="50" velocity="50" lower="0" upper="0" />
+      <dynamics damping="0.0" friction="10"/>
+    </joint>
+  <gazebo>
+      <plugin name="gazebo_ros_vacuum_gripper1" filename="libgazebo_ros_vacuum_gripper.so">
+        <robotNamespace>/ur5/vacuum_gripper1</robotNamespace>
+        <bodyName>vacuum_gripper1</bodyName>
+        <topicName>grasping1</topicName>
+	<maxForce>50</maxForce>
+        <maxDistance>0.05</maxDistance>
+        <minDistance>0.01</minDistance>
+      </plugin>
+  </gazebo>
+    <link name="vacuum_gripper2">
+      <gravity>0</gravity>
+      <visual>
+        <origin rpy="0 0 0" xyz="0 0 0"/>
+        <geometry>
+          <cylinder radius="0.005" length="0.01"/>
+        </geometry>
+        <material name="transparent">
+          <color rgba="0 0 0 0"/>
+        </material>
+      </visual>
+      <inertial>
+        <origin rpy="0 0 0" xyz="0.000000 0.000000 0.000000"/>
+        <mass value="0.0001"/>
+        <inertia ixx="1e-08" ixy="0" ixz="0" iyy="1e-08" iyz="0" izz="1e-08"/>
+      </inertial>
+    </link>
+    <joint name="gripper_joint2" type="revolute">
+      <axis xyz="1 0 0" />
+      <parent link="ee_link" />
+      <child link="vacuum_gripper2" />
+      <origin rpy="0 1.5708 0" xyz="0.01 0 0.0125" />
+      <limit effort="50" velocity="50" lower="0" upper="0" />
+      <dynamics damping="0.0" friction="10"/>
+    </joint>
+  <gazebo>
+      <plugin name="gazebo_ros_vacuum_gripper2" filename="libgazebo_ros_vacuum_gripper.so">
+        <robotNamespace>/ur5/vacuum_gripper2</robotNamespace>
+        <bodyName>vacuum_gripper2</bodyName>
+        <topicName>grasping2</topicName>
+	<maxForce>50</maxForce>
+        <maxDistance>0.05</maxDistance>
+        <minDistance>0.01</minDistance>
+      </plugin>
+  </gazebo>
+    <link name="vacuum_gripper3">
+      <gravity>0</gravity>
+      <visual>
+        <origin rpy="0 0 0" xyz="0 0 0"/>
+        <geometry>
+          <cylinder radius="0.005" length="0.01"/>
+        </geometry>
+        <material name="transparent">
+          <color rgba="0 0 0 0"/>
+        </material>
+      </visual>
+      <inertial>
+        <origin rpy="0 0 0" xyz="0.000000 0.000000 0.000000"/>
+        <mass value="0.0001"/>
+        <inertia ixx="1e-08" ixy="0" ixz="0" iyy="1e-08" iyz="0" izz="1e-08"/>
+      </inertial>
+    </link>
+    <joint name="gripper_joint3" type="revolute">
+      <axis xyz="1 0 0" />
+      <parent link="ee_link" />
+      <child link="vacuum_gripper3" />
+      <origin rpy="0 1.5708 0" xyz="0.01 0 -0.0125" />
+      <limit effort="50" velocity="50" lower="0" upper="0" />
+      <dynamics damping="0.0" friction="10"/>
+    </joint>
+  <gazebo>
+      <plugin name="gazebo_ros_vacuum_gripper3" filename="libgazebo_ros_vacuum_gripper.so">
+        <robotNamespace>/ur5/vacuum_gripper3</robotNamespace>
+        <bodyName>vacuum_gripper3</bodyName>
+        <topicName>grasping2</topicName>
+	<maxForce>50</maxForce>
+        <maxDistance>0.05</maxDistance>
+        <minDistance>0.01</minDistance>
+      </plugin>
+  </gazebo>
+  <link name="vacuum_gripper4">
+    <gravity>0</gravity>
+    <visual>
+      <origin rpy="0 0 0" xyz="0 0 0"/>
+      <geometry>
+        <cylinder radius="0.005" length="0.01"/>
+      </geometry>
+      <material name="transparent">
+        <color rgba="0 0 0 0"/>
+      </material>
+    </visual>
+    <inertial>
+      <origin rpy="0 0 0" xyz="0.000000 0.000000 0.000000"/>
+      <mass value="0.0001"/>
+      <inertia ixx="1e-08" ixy="0" ixz="0" iyy="1e-08" iyz="0" izz="1e-08"/>
+    </inertial>
+  </link>
+  <joint name="gripper_joint4" type="revolute">
+    <axis xyz="1 0 0" />
+    <parent link="ee_link" />
+    <child link="vacuum_gripper4" />
+    <origin rpy="0 1.5708 0" xyz="0.01 0 0" />
+    <limit effort="50" velocity="50" lower="0" upper="0" />
+    <dynamics damping="0.0" friction="10"/>
+  </joint>
+  <gazebo>
+    <plugin name="gazebo_ros_vacuum_gripper4" filename="libgazebo_ros_vacuum_gripper.so">
+      <robotNamespace>/ur5/vacuum_gripper4</robotNamespace>
+      <bodyName>vacuum_gripper4</bodyName>
+      <topicName>grasping4</topicName>
+  <maxForce>50</maxForce>
+      <maxDistance>0.05</maxDistance>
+      <minDistance>0.01</minDistance>
+    </plugin>
+  </gazebo>
+  <link name="vacuum_gripper5">
+    <gravity>0</gravity>
+    <visual>
+      <origin rpy="0 0 0" xyz="0 0 0"/>
+      <geometry>
+        <cylinder radius="0.005" length="0.01"/>
+      </geometry>
+      <material name="transparent">
+        <color rgba="0 0 0 0"/>
+      </material>
+    </visual>
+    <inertial>
+      <origin rpy="0 0 0" xyz="0.000000 0.000000 0.000000"/>
+      <mass value="0.0001"/>
+      <inertia ixx="1e-08" ixy="0" ixz="0" iyy="1e-08" iyz="0" izz="1e-08"/>
+    </inertial>
+  </link>
+  <joint name="gripper_joint5" type="revolute">
+    <axis xyz="1 0 0" />
+    <parent link="ee_link" />
+    <child link="vacuum_gripper5" />
+    <origin rpy="0 1.5708 0" xyz="0.01 0.0125 0.0125" />
+    <limit effort="50" velocity="50" lower="0" upper="0" />
+    <dynamics damping="0.0" friction="10"/>
+  </joint>
+<gazebo>
+    <plugin name="gazebo_ros_vacuum_gripper" filename="libgazebo_ros_vacuum_gripper.so">
+      <robotNamespace>/ur5/vacuum_gripper5</robotNamespace>
+      <bodyName>vacuum_gripper5</bodyName>
+      <topicName>grasping5</topicName>
+<maxForce>50</maxForce>
+      <maxDistance>0.05</maxDistance>
+      <minDistance>0.01</minDistance>
+    </plugin>
+</gazebo>
+  <link name="vacuum_gripper6">
+    <gravity>0</gravity>
+    <visual>
+      <origin rpy="0 0 0" xyz="0 0 0"/>
+      <geometry>
+        <cylinder radius="0.005" length="0.01"/>
+      </geometry>
+      <material name="transparent">
+        <color rgba="0 0 0 0"/>
+      </material>
+    </visual>
+    <inertial>
+      <origin rpy="0 0 0" xyz="0.000000 0.000000 0.000000"/>
+      <mass value="0.0001"/>
+      <inertia ixx="1e-08" ixy="0" ixz="0" iyy="1e-08" iyz="0" izz="1e-08"/>
+    </inertial>
+  </link>
+  <joint name="gripper_joint6" type="revolute">
+    <axis xyz="1 0 0" />
+    <parent link="ee_link" />
+    <child link="vacuum_gripper6" />
+    <origin rpy="0 1.5708 0" xyz="0.01 -0.0125 0.0125" />
+    <limit effort="50" velocity="50" lower="0" upper="0" />
+    <dynamics damping="0.0" friction="10"/>
+  </joint>
+<gazebo>
+    <plugin name="gazebo_ros_vacuum_gripper1" filename="libgazebo_ros_vacuum_gripper.so">
+      <robotNamespace>/ur5/vacuum_gripper6</robotNamespace>
+      <bodyName>vacuum_gripper6</bodyName>
+      <topicName>grasping6</topicName>
+<maxForce>50</maxForce>
+      <maxDistance>0.05</maxDistance>
+      <minDistance>0.01</minDistance>
+    </plugin>
+</gazebo>
+  <link name="vacuum_gripper7">
+    <gravity>0</gravity>
+    <visual>
+      <origin rpy="0 0 0" xyz="0 0 0"/>
+      <geometry>
+        <cylinder radius="0.005" length="0.01"/>
+      </geometry>
+      <material name="transparent">
+        <color rgba="0 0 0 0"/>
+      </material>
+    </visual>
+    <inertial>
+      <origin rpy="0 0 0" xyz="0.000000 0.000000 0.000000"/>
+      <mass value="0.0001"/>
+      <inertia ixx="1e-08" ixy="0" ixz="0" iyy="1e-08" iyz="0" izz="1e-08"/>
+    </inertial>
+  </link>
+  <joint name="gripper_joint7" type="revolute">
+    <axis xyz="1 0 0" />
+    <parent link="ee_link" />
+    <child link="vacuum_gripper7" />
+    <origin rpy="0 1.5708 0" xyz="0.01 0.0125 -0.0125" />
+    <limit effort="50" velocity="50" lower="0" upper="0" />
+    <dynamics damping="0.0" friction="10"/>
+  </joint>
+<gazebo>
+    <plugin name="gazebo_ros_vacuum_gripper7" filename="libgazebo_ros_vacuum_gripper.so">
+      <robotNamespace>/ur5/vacuum_gripper7</robotNamespace>
+      <bodyName>vacuum_gripper7</bodyName>
+      <topicName>grasping7</topicName>
+<maxForce>50</maxForce>
+      <maxDistance>0.05</maxDistance>
+      <minDistance>0.01</minDistance>
+    </plugin>
+</gazebo>
+  <link name="vacuum_gripper8">
+    <gravity>0</gravity>
+    <visual>
+      <origin rpy="0 0 0" xyz="0 0 0"/>
+      <geometry>
+        <cylinder radius="0.005" length="0.01"/>
+      </geometry>
+      <material name="transparent">
+        <color rgba="0 0 0 0"/>
+      </material>
+    </visual>
+    <inertial>
+      <origin rpy="0 0 0" xyz="0.000000 0.000000 0.000000"/>
+      <mass value="0.0001"/>
+      <inertia ixx="1e-08" ixy="0" ixz="0" iyy="1e-08" iyz="0" izz="1e-08"/>
+    </inertial>
+  </link>
+  <joint name="gripper_joint8" type="revolute">
+    <axis xyz="1 0 0" />
+    <parent link="ee_link" />
+    <child link="vacuum_gripper8" />
+    <origin rpy="0 1.5708 0" xyz="0.01 -0.0125 -0.0125" />
+    <limit effort="50" velocity="50" lower="0" upper="0" />
+    <dynamics damping="0.0" friction="10"/>
+  </joint>
+<gazebo>
+    <plugin name="gazebo_ros_vacuum_gripper8" filename="libgazebo_ros_vacuum_gripper.so">
+      <robotNamespace>/ur5/vacuum_gripper8</robotNamespace>
+      <bodyName>vacuum_gripper8</bodyName>
+      <topicName>grasping8</topicName>
+<maxForce>50</maxForce>
+      <maxDistance>0.05</maxDistance>
+      <minDistance>0.01</minDistance>
+    </plugin>
+</gazebo>
   <link name="camera_mount_1">
     <inertial>
